Commit message: Finished model plagin 3d lidar

File: src/turtlebot3/turtlebot3_description/urdf/turtlebot3_my_burger.gazebo.xacro (robot description, xacro)
@@ -97,5 +97,5 @@
         <sensor type="ray" name="sensor">
             <always_on>true</always_on>
-            <pose>0 0 -0.004645 1.5707 0 0</pose>
+            <pose>0 0 0.04 1.5707 0 0</pose>
             <visualize>true</visualize>
             <ray>

File: src/turtlebot3/turtlebot3_description/urdf/turtlebot3_my_burger.urdf.xacro (robot description, xacro)
@@ -119,10 +119,10 @@
         <parent link="base_link"/>
         <child link="base_lidar"/>
-        <origin xyz="-0.032 0 0.172" rpy="0 0 0"/>
+        <origin xyz="-0.022519 0.002564 0.140612" rpy="0 0 0"/>
     </joint>
     <link name="base_lidar">
-        <pose>0 0 0.029335 0 0 0</pose>
+        <origin xyz="0 0 0.029335" rpy="0 0 0"/>
         <inertial>
-            <mass value="1.2"/>
+            <mass value="0.2"/>
             <inertia ixx="0.001087473" ixy="0" ixz="0" iyy="0.001087473" iyz="0" izz="0.001092437"/>
         </inertial>
@@ -132,13 +132,13 @@
             </geometry>
         </collision>
-        <!--        <visual name="base_visual">-->
-        <!--            <pose>0 0 -0.029335 0 0 0</pose>-->
-        <!--            <geometry>-->
-        <!--                <mesh filename="model://velodyne_hdl32/meshes/velodyne_base.dae"/>-->
-        <!--            </geometry>-->
-        <!--        </visual>-->
+        <visual name="base_visual">
+            <pose>0 0 -0.029335 0 0 0</pose>
+            <geometry>
+                <mesh filename="model://velodyne_hdl32/meshes/velodyne_base.dae"/>
+            </geometry>
+        </visual>
     </link>
     <link name="top_lidar">
-        <pose>0 0 0.095455 0 0 0</pose>
+        <origin rpy="0 0 0" xyz="0 0 0.095455"/>
         <inertial>
             <mass value="0.1"/>
@@ -158,5 +158,5 @@
     </link>
     <joint type="revolute" name="velodyne_joint">
-        <pose>0 0 -0.036785 0 0 0</pose>
+        <origin xyz="0 0 0.056785" rpy="0 0 0"/>
         <parent link="base_lidar"/>
         <child link="top_lidar"/>

Commit message: tmp commit

File: src/turtlebot3/turtlebot3_description/urdf/turtlebot3_my_burger.gazebo.xacro (robot description, xacro)
@@ -97,5 +97,5 @@
         <sensor type="ray" name="sensor">
             <always_on>true</always_on>
-            <pose>0 0 0.04 1.5707 0 0</pose>
+            <pose>0 0 0.04 1.5707 0 -1.6</pose>
             <visualize>true</visualize>
             <ray>
@@ -123,7 +123,8 @@
     </gazebo>
     <gazebo>
-        <plugin name="velodyne_control" filename="libvelodyne_plugin.so">
-            <velocity>25</velocity>
-        </plugin>
+<!--        <plugin name="velodyne_model_control" filename="libvelodyne_model_plugin.so">-->
+<!--            <rotate_speed>0</rotate_speed>-->
+<!--        </plugin>-->
+        <plugin name="velodyne_sensor_control" filename="libvelodyne_sensor_plugin.so"/>
     </gazebo>
     <!--link : https://www.raspberrypi.org/documentation/hardware/camera/-->

File: src/turtlebot3/turtlebot3_description/urdf/turtlebot3_my_burger.urdf.xacro (robot description, xacro)
@@ -119,5 +119,5 @@
         <parent link="base_link"/>
         <child link="base_lidar"/>
-        <origin xyz="-0.022519 0.002564 0.140612" rpy="0 0 0"/>
+        <origin xyz="-0.022519 0 0.140612" rpy="0 0 0"/>
     </joint>
     <link name="base_lidar">
@@ -158,9 +158,9 @@
     </link>
     <joint type="revolute" name="velodyne_joint">
-        <origin xyz="0 0 0.056785" rpy="0 0 0"/>
+        <origin xyz="0 0 0.056785" rpy="0 0 1.5707"/>
         <parent link="base_lidar"/>
         <child link="top_lidar"/>
         <axis xyz="0 0 1"/>
-        <limit effort="10" velocity="10" lower="-10000000000000000" upper="10000000000000000"/>
+        <limit effort="1" velocity="1000000" lower="-10000000000000000" upper="10000000000000000"/>
     </joint>
     <joint name="camera_joint" type="fixed">
