Commit message: Changed lidar model config

File: src/turtlebot3/turtlebot3_description/urdf/turtlebot3_my_burger.urdf.xacro (robot description, xacro)
@@ -124,6 +124,6 @@
         <origin xyz="0 0 0.029335" rpy="0 0 0"/>
         <inertial>
-            <mass value="0.2"/>
-            <inertia ixx="0.001087473" ixy="0" ixz="0" iyy="0.001087473" iyz="0" izz="0.001092437"/>
+            <mass value="0.02"/>
+            <inertia ixx="0.0001087473" ixy="0" ixz="0" iyy="0.0001087473" iyz="0" izz="0.0001092437"/>
         </inertial>
         <collision name="base_collision">
@@ -142,6 +142,6 @@
         <origin rpy="0 0 0" xyz="0 0 0.095455"/>
         <inertial>
-            <mass value="0.1"/>
-            <inertia ixx="0.000090623" izz="0.000091036" iyy="0.000090623" iyz="0" ixz="0" ixy="0"/>
+            <mass value="0.01"/>
+            <inertia ixx="0.0000090623" izz="0.000091036" iyy="0.0000090623" iyz="0" ixz="0" ixy="0"/>
         </inertial>
         <collision name="top_collision">
